File: schematics/fan_control_circuit/_autosave-fan_control_circuit.kicad_sch (KiCad schematic)
At the start: 32 parts, among them U1 RASPBERRY_PI_4B_4GB, U2 BME280, U3 SHT30-DIS, U4 STM32F103C8Tx, U5 TMP36xS

Commit message: schematics
Changed lines of the file:
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@@
-	)
-	(junction
-		(at 220.98 72.39)
-		(diameter 0)
-		(color 0 0 0 0)
 	)
 	(junction
@@
 	)
 	(junction
-		(at 234.95 95.25)
+		(at 248.92 95.25)
 		(diameter 0)
 		(color 0 0 0 0)
@@
 	)
 	(junction
-		(at 214.63 119.38)
+		(at 227.33 72.39)
 		(diameter 0)
 		(color 0 0 0 0)
@@
 	)
 	(junction
+		(at 205.74 119.38)
+		(diameter 0)
+		(color 0 0 0 0)
+	)
+	(junction
 		(at 250.19 69.85)
 		(diameter 0)
@@
 	(wire
 		(pts
-			(xy 200.66 119.38) (xy 214.63 119.38)
+			(xy 200.66 119.38) (xy 205.74 119.38)
 		)
 		(stroke
@@
 	(wire
 		(pts
-			(xy 220.98 69.85) (xy 220.98 72.39)
+			(xy 227.33 69.85) (xy 227.33 72.39)
 		)
 		(stroke
@@
 	(wire
 		(pts
-			(xy 234.95 90.17) (xy 234.95 95.25)
+			(xy 248.92 90.17) (xy 248.92 95.25)
 		)
 		(stroke
@@
 	(wire
 		(pts
-			(xy 214.63 119.38) (xy 237.49 119.38)
-		)
-		(stroke
-			(width 0)
-			(type default)
-		)
-	)
-	(wire
-		(pts
 			(xy 278.13 143.51) (xy 278.13 156.21)
 		)
@@
 	(wire
 		(pts
-			(xy 214.63 72.39) (xy 220.98 72.39)
+			(xy 214.63 72.39) (xy 227.33 72.39)
 		)
 		(stroke
@@
 	(wire
 		(pts
+			(xy 248.92 95.25) (xy 264.16 95.25)
+		)
+		(stroke
+			(width 0)
+			(type default)
+		)
+	)
+	(wire
+		(pts
 			(xy 15.24 160.02) (xy 15.24 154.94)
 		)
@@
 	(wire
 		(pts
-			(xy 234.95 95.25) (xy 242.57 95.25)
-		)
-		(stroke
-			(width 0)
-			(type default)
-		)
-	)
-	(wire
-		(pts
-			(xy 242.57 95.25) (xy 264.16 95.25)
-		)
-		(stroke
-			(width 0)
-			(type default)
-		)
-	)
-	(wire
-		(pts
 			(xy 195.58 129.54) (xy 195.58 46.99)
 		)
@@
 	(wire
 		(pts
+			(xy 205.74 92.71) (xy 214.63 92.71)
+		)
+		(stroke
+			(width 0)
+			(type default)
+		)
+	)
+	(wire
+		(pts
 			(xy 242.57 67.31) (xy 261.62 67.31)
 		)
@@
 	(wire
 		(pts
+			(xy 248.92 95.25) (xy 242.57 95.25)
+		)
+		(stroke
+			(width 0)
+			(type default)
+		)
+	)
+	(wire
+		(pts
 			(xy 267.97 143.51) (xy 278.13 143.51)
 		)
@@
 	(wire
 		(pts
-			(xy 220.98 69.85) (xy 250.19 69.85)
+			(xy 227.33 69.85) (xy 250.19 69.85)
 		)
 		(stroke
@@
 	(wire
 		(pts
-			(xy 250.19 90.17) (xy 234.95 90.17)
+			(xy 250.19 90.17) (xy 248.92 90.17)
 		)
 		(stroke
@@
 	(wire
 		(pts
-			(xy 203.2 95.25) (xy 234.95 95.25)
+			(xy 203.2 95.25) (xy 242.57 95.25)
 		)
 		(stroke
@@
 	(wire
 		(pts
+			(xy 205.74 119.38) (xy 237.49 119.38)
+		)
+		(stroke
+			(width 0)
+			(type default)
+		)
+	)
+	(wire
+		(pts
 			(xy 198.12 39.37) (xy 198.12 127)
 		)
@@
 	(wire
 		(pts
-			(xy 220.98 72.39) (xy 227.33 72.39)
-		)
-		(stroke
-			(width 0)
-			(type default)
-		)
-	)
-	(wire
-		(pts
 			(xy 227.33 72.39) (xy 227.33 74.93)
 		)
@@
 	(wire
 		(pts
-			(xy 214.63 92.71) (xy 214.63 119.38)
-		)
-		(stroke
+			(xy 205.74 92.71) (xy 205.74 119.38)
+		)
+		(stroke
