File: schematics/fan_control_circuit/my_piHAT_v1.kicad_sch (KiCad schematic)
At the start: 32 parts, among them U1 RASPBERRY_PI_4B_4GB, U2 BME280, U3 SHT30-DIS, U4 STM32F103C8Tx, U5 TMP36xS

Commit message: schematics
Parts:
- removed C?: 0.1uF, Capacitor_SMD:CP_Elec_3x5.3, symbol Device:C_Polarized_Small_US
- removed D?: CLEAR(TX), LED_SMD:LED-APA102-2020, symbol Device:LED
- removed Q? (x2): 2N3904, Package_TO_SOT_THT:TO-92_Inline, symbol Transistor_BJT:2N3904
- removed R? (x2): 4.7k, OptoDevice:R_LDR_4.9x4.2mm_P2.54mm_Vertical, symbol Device:R
- removed R?: 110, OptoDevice:R_LDR_4.9x4.2mm_P2.54mm_Vertical, symbol Device:R
- removed R?: 1m, OptoDevice:R_LDR_4.9x4.2mm_P2.54mm_Vertical, symbol Device:R
- removed R?: 10k, OptoDevice:R_LDR_4.9x4.2mm_P2.54mm_Vertical, symbol Device:R
- removed U?: ~, symbol my_parts:MQ-6-FF
- added U?: MQ-6, Sensor:MQ-6, symbol Sensor_Gas:MQ-6
- C?: value 10uF -> 470uF
Connections:
- net COM: no longer C?.1
- net at F1.2 (-), F2.2 (-), U4.23 (VSS_1)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: no longer C?.2
Other:
- moved on the sheet: C?, F2, Q?, U?
