File: schematics/fan_control_circuit/fan_control_circuit.kicad_sch (KiCad schematic)
At the start: 32 parts, among them U1 RASPBERRY_PI_4B_4GB, U2 BME280, U3 SHT30-DIS, U4 STM32F103C8Tx, U5 TMP36xS

Commit message: schematic
Other:
- moved on the sheet: C?, U?
